File: CAD/Sustainer/av bay ideas/sled/sled.kicad_sch (KiCad schematic)
At the start: 23 parts, among them J1 Conn_01x02, J2 Conn_01x02, SW1 SW_DIP_x01, SW2 SW_DIP_x01, SW3 SW_DIP_x01, SW4 SW_DIP_x01

Commit message: new sled
Parts:
- removed H7: MountingHole_Pad, MountingHole:MountingHole_2.2mm_M2_DIN965_Pad, symbol Mechanical:MountingHole_Pad
- removed J1: Conn_01x02, Connector_PinHeader_2.54mm:PinHeader_1x02_P2.54mm_Vertical, symbol Connector_Generic:Conn_01x02
- added D1, D2, D3: LED, LED_SMD:LED_0603_1608Metric, symbol Device:LED
- added R1, R2, R3: 1k, Resistor_SMD:R_0603_1608Metric, symbol Device:R_Small
- added SW5: SW_SPDT, TerminalBlock:TerminalBlock_bornier-3_P5.08mm, symbol Switch:SW_SPDT
Connections:
- net BR_NEG: now also D2.1 (K)
- net BR_POS: now also SW5.3 (C)
- net HEI: now also SW5.2 (B)
- net at BT2.2 (-), LYRA1.1 (BATT-): now also D1.1 (K)
- net at BT2.1 (+), LYRA1.2 (BATT+): now also R1.2
- net at GPS1.2 (VIN), SW3.2: now also R3.2
- net at BT3.2 (-), GPS1.1 (GND): now also D3.1 (K)
- net at BT1.1 (+), SW1.1: now also R2.2
- new net: D2.2 (A), R2.1
- new net: D1.2 (A), R1.1
- new net: D3.2 (A), R3.1
- no-connect marks 12 -> 13
Other:
- moved on the sheet: GPS1, SW2
