File: CAD/Sustainer/av bay silicdyne please/aftbulkhead/aftbulkhead.kicad_pcb (KiCad board)
At the start: 2 copper layers, 30.7 x 30.7 mm, 11 parts, among them J1 Conn_01x02, SW1 SW_SPDT

Commit message: work
Parts:
- removed H2: MountingHole, MountingHole:MountingHole_2.2mm_M2
- removed J1: Conn_01x02, Connector_PinHeader_2.54mm:PinHeader_1x02_P2.54mm_Vertical
- removed SW1: SW_SPDT, TerminalBlock:TerminalBlock_bornier-3_P5.08mm
- added REF**: PinHeader_1x05_P2.54mm_Vertical, Connector_PinHeader_2.54mm:PinHeader_1x05_P2.54mm_Vertical, F.Cu at (163.5, 80.2)
- moved H1 2.55 mm to (158.0, 90.2)
- moved H3 0.28 mm to (158.0, 80.0)
Routing:
- net Net-(J1-Pin_2): track 17.5 -> 0.00 mm
- net Net-(J1-Pin_1): track 15.1 -> 0.00 mm
Other:
- outline, holes or cut-outs redrawn
