File: CAD/Sustainer/av bay silicdyne please/sled/sled.kicad_sch (KiCad schematic)
At the start: 28 parts, among them J2 Conn_01x02, SW1 SW_DIP_x01, SW2 SW_DIP_x01, SW3 SW_DIP_x01, SW4 SW_DIP_x01, SW5 SW_SPDT

Commit message: work
Parts:
- removed BR1: ~, Connector_PinHeader_2.54mm:PinHeader_1x06_P2.54mm_Vertical, symbol Altimeters:Blue_Raven
- removed BT1: Battery, Connector_PinHeader_1.27mm:PinHeader_1x02_P1.27mm_Vertical, symbol Device:Battery
- removed D3: LED, LED_SMD:LED_0603_1608Metric, symbol Device:LED
- removed GPS1: ~, Connector_PinHeader_2.54mm:PinHeader_1x02_P2.54mm_Vertical, symbol Altimeters:Featherweight GPS
- removed H10, H6: MountingHole_Pad, MountingHole:MountingHole_2.2mm_M2_DIN965_Pad, symbol Mechanical:MountingHole_Pad
- removed R3: 1k, Resistor_SMD:R_0603_1608Metric, symbol Device:R_Small
- removed SW3: SW_DIP_x01, Connector_PinHeader_2.54mm:PinHeader_2x01_P2.54mm_Horizontal, symbol Switch:SW_DIP_x01
- removed SW4: SW_DIP_x01, Connector_PinHeader_2.54mm:PinHeader_1x01_P2.54mm_Horizontal, symbol Switch:SW_DIP_x01
- added J1: Conn_01x02, Connector_PinHeader_2.54mm:PinHeader_1x02_P2.54mm_Vertical, symbol Connector_Generic:Conn_01x02
- added J3: Conn_01x04, .pretty:4 pads 2.54mm spacign, symbol Connector_Generic:Conn_01x04
- BT3: footprint easyeda2kicad:CONN-TH_2P-P2.00_PH-2AK -> Connector_JST:JST_PH_B2B-PH-K_1x02_P2.00mm_Vertical
- H1, H2, H3, H5: footprint MountingHole:MountingHole_3.2mm_M3_Pad -> MountingHole:MountingHole_3.2mm_M3
- H4: footprint MountingHole:MountingHole_3.2mm_M3_Pad -> MountingHole:MountingHole_2.2mm_M2_DIN965_Pad
- SW1, SW2: footprint Connector_PinHeader_2.54mm:PinHeader_2x01_P2.54mm_Horizontal -> Connector_PinHeader_2.54mm:PinHeader_1x02_P2.54mm_Vertical
Connections:
- net BR_NEG is gone; now on net FLUCTUS NEG: D2.1 (K)
- net APOGEE: now also H4.1, J3.1 (Pin_1)
- net HEI: now also J3.3 (Pin_3)
- net MAIN: now also J3.2 (Pin_2)
- net at BT3.1 (+): now also R2.2, SW1.1
- net FLUCTUS NEG: now reaches BT3.2 (-)
- net FLUCTUS NEG: now also J1.1 (Pin_1)
- net BR_POS renamed PYRO POS
- net PYRO POS: now also J3.4 (Pin_4); no longer SW1.2
- new net FLUCTUS POS: J1.2 (Pin_2), SW1.2
- no-connect marks 13 -> 14
Other:
- moved on the sheet: H11, SW5
